File: sample-board.kicad_sch (KiCad schematic)
At the start: 0 parts

Commit message: Test board: LED Blinker
Parts:
- added C1: 10uC, Capacitor_THT:C_Disc_D5.0mm_W2.5mm_P2.50mm, symbol Device:C
- added C2: 0.01uC, Capacitor_THT:C_Disc_D5.0mm_W2.5mm_P2.50mm, symbol Device:C
- added D1: LED, LED_THT:LED_D3.0mm, symbol Device:LED
- added J2: USB_B_Micro, Connector_USB:USB_Micro-AB_Molex_47590-0001, symbol Connector:USB_B_Micro
- added R1: 1kR, Resistor_THT:R_Axial_DIN0207_L6.3mm_D2.5mm_P2.54mm_Vertical, symbol Device:R
- added R2: 10kR, Resistor_THT:R_Axial_DIN0207_L6.3mm_D2.5mm_P2.54mm_Vertical, symbol Device:R
- added R3: 220R, Resistor_THT:R_Axial_DIN0207_L6.3mm_D2.5mm_P2.54mm_Vertical, symbol Device:R
- added U1: LM555xN, Package_DIP:DIP-8_W7.62mm, symbol Timer:LM555xN
Connections:
- new net: R3.1, U1.3 (OUT)
- new net: D1.2 (A), R3.2
- new net: R1.2, R2.1, U1.7 (DISCH)
- new net: C1.1, R2.2, U1.2 (TRIG), U1.6 (THRES)
- new net: J2.1 (VBUS), R1.1, U1.4 (~{RST}), U1.8 (VCC)
- new net: C1.2, C2.2, D1.1 (K), J2.5 (GND), U1.1 (GND)
- new net: C2.1, U1.5 (CONT)
- no-connect marks 0 -> 4
